Commit message: add a1 elements

File: meshes/a1/urdf/a1.urdf.xacro (robot description, xacro)
@@ -115,18 +115,4 @@
     </inertial>
   </link>
-  <joint name="fr_fixed_j0" type="fixed">
-    <origin rpy="0 0 0" xyz="0 -0.081 0"/>
-    <parent link="fr_l0"/>
-    <child link="fr_l0_shoulder"/>
-  </joint>
-  <!-- this link is only for collision -->
-  <link name="fr_l0_shoulder">
-    <!-- <collision>
-      <origin rpy="1.57079632679 0 0" xyz="0 0 0"/>
-      <geometry>
-        <cylinder length="0.032" radius="0.041"/>
-      </geometry>
-    </collision> -->
-  </link>
   <joint name="fr_j1" type="revolute">
     <origin rpy="0 0 0" xyz="0 -0.08505 0"/>
@@ -157,5 +143,5 @@
     </inertial>
   </link>
-  <joint name="fr_j1" type="revolute">
+  <joint name="fr_j2" type="revolute">
     <origin rpy="0 0 0" xyz="0 0 -0.2"/>
     <parent link="fr_l1"/>
@@ -209,13 +195,13 @@
     </inertial>
   </link>
-  <joint name="FL_hip_joint" type="revolute">
+  <joint name="fl_j0" type="revolute">
     <origin rpy="0 0 0" xyz="0.183 0.047 0"/>
     <parent link="trunk"/>
-    <child link="FL_hip"/>
+    <child link="fl_l0"/>
     <axis xyz="1 0 0"/>
     <dynamics damping="0" friction="0"/>
     <limit effort="20" lower="-0.802851455917" upper="0.802851455917" velocity="52.4"/>
   </joint>
-  <link name="FL_hip">
+  <link name="fl_l0">
     <visual>
       <origin rpy="0 0 0" xyz="0 0 0"/>
@@ -237,27 +223,13 @@
     </inertial>
   </link>
-  <joint name="FL_hip_fixed" type="fixed">
-    <origin rpy="0 0 0" xyz="0 0.081 0"/>
-    <parent link="FL_hip"/>
-    <child link="FL_thigh_shoulder"/>
-  </joint>
-  <!-- this link is only for collision -->
-  <link name="FL_thigh_shoulder">
-    <!-- <collision>
-      <origin rpy="1.57079632679 0 0" xyz="0 0 0"/>
-      <geometry>
-        <cylinder length="0.032" radius="0.041"/>
-      </geometry>
-    </collision> -->
-  </link>
-  <joint name="FL_thigh_joint" type="revolute">
+  <joint name="fl_j1" type="revolute">
     <origin rpy="0 0 0" xyz="0 0.08505 0"/>
-    <parent link="FL_hip"/>
-    <child link="FL_thigh"/>
+    <parent link="fl_l0"/>
+    <child link="fl_l1"/>
     <axis xyz="0 1 0"/>
     <dynamics damping="0" friction="0"/>
     <limit effort="55" lower="-1.0471975512" upper="4.18879020479" velocity="28.6"/>
   </joint>
-  <link name="FL_thigh">
+  <link name="fl_l1">
     <visual>
       <origin rpy="0 0 0" xyz="0 0 0"/>
@@ -279,13 +251,13 @@
     </inertial>
   </link>
-  <joint name="FL_calf_joint" type="revolute">
-    <origin rpy="0 0 0" xyz="0 0 -0.2"/>
-    <parent link="FL_thigh"/>
-    <child link="FL_calf"/>
+  <joint name="fl_j2" type="revolute">
+    <origin rpy="0 0 0" xyz="0 0 -0.2"/>
+    <parent link="fl_l1"/>
+    <child link="fl_l2"/>
     <axis xyz="0 1 0"/>
     <dynamics damping="0" friction="0"/>
     <limit effort="55" lower="-2.69653369433" upper="-0.916297857297" velocity="28.6"/>
   </joint>
-  <link name="FL_calf">
+  <link name="fl_l2">
     <visual>
       <origin rpy="0 0 0" xyz="0 0 0"/>
@@ -307,10 +279,10 @@
     </inertial>
   </link>
-  <joint name="FL_foot_fixed" type="fixed" dont_collapse="true">
-    <origin rpy="0 0 0" xyz="0 0 -0.2"/>
-    <parent link="FL_calf"/>
-    <child link="FL_foot"/>
-  </joint>
-  <link name="FL_foot">
+  <joint name="fl_j3" type="fixed" dont_collapse="true">
+    <origin rpy="0 0 0" xyz="0 0 -0.2"/>
+    <parent link="fl_l2"/>
+    <child link="fl_l3"/>
+  </joint>
+  <link name="fl_l3">
     <visual>
       <origin rpy="0 0 0" xyz="0 0 0"/>
@@ -331,13 +303,13 @@
     </inertial>
   </link>
-  <joint name="RR_hip_joint" type="revolute">
+  <joint name="rr_j0" type="revolute">
     <origin rpy="0 0 0" xyz="-0.183 -0.047 0"/>
     <parent link="trunk"/>
-    <child link="RR_hip"/>
+    <child link="rr_l0"/>
     <axis xyz="1 0 0"/>
     <dynamics damping="0" friction="0"/>
     <limit effort="20" lower="-0.802851455917" upper="0.802851455917" velocity="52.4"/>
   </joint>
-  <link name="RR_hip">
+  <link name="rr_l0">
     <visual>
       <origin rpy="3.14159265359 3.14159265359 0" xyz="0 0 0"/>
@@ -359,27 +331,13 @@
     </inertial>
   </link>
-  <joint name="RR_hip_fixed" type="fixed">
-    <origin rpy="0 0 0" xyz="0 -0.081 0"/>
-    <parent link="RR_hip"/>
-    <child link="RR_thigh_shoulder"/>
-  </joint>
-  <!-- this link is only for collision -->
-  <link name="RR_thigh_shoulder">
-    <!-- <collision>
-      <origin rpy="1.57079632679 0 0" xyz="0 0 0"/>
-      <geometry>
-        <cylinder length="0.032" radius="0.041"/>
-      </geometry>
-    </collision> -->
-  </link>
-  <joint name="RR_thigh_joint" type="revolute">
+  <joint name="rr_j1" type="revolute">
     <origin rpy="0 0 0" xyz="0 -0.08505 0"/>
-    <parent link="RR_hip"/>
-    <child link="RR_thigh"/>
+    <parent link="rr_l0"/>
+    <child link="rr_l1"/>
     <axis xyz="0 1 0"/>
     <dynamics damping="0" friction="0"/>
     <limit effort="55" lower="-1.0471975512" upper="4.18879020479" velocity="28.6"/>
   </joint>
-  <link name="RR_thigh">
+  <link name="rr_l1">
     <visual>
       <origin rpy="0 0 0" xyz="0 0 0"/>
@@ -401,13 +359,13 @@
     </inertial>
   </link>
-  <joint name="RR_calf_joint" type="revolute">
-    <origin rpy="0 0 0" xyz="0 0 -0.2"/>
-    <parent link="RR_thigh"/>
-    <child link="RR_calf"/>
+  <joint name="rr_j2" type="revolute">
+    <origin rpy="0 0 0" xyz="0 0 -0.2"/>
+    <parent link="rr_l1"/>
+    <child link="rr_l2"/>
     <axis xyz="0 1 0"/>
     <dynamics damping="0" friction="0"/>
     <limit effort="55" lower="-2.69653369433" upper="-0.916297857297" velocity="28.6"/>
   </joint>
-  <link name="RR_calf">
+  <link name="rr_l2">
     <visual>
       <origin rpy="0 0 0" xyz="0 0 0"/>
@@ -429,10 +387,10 @@
     </inertial>
   </link>
-  <joint name="RR_foot_fixed" type="fixed" dont_collapse="true">
-    <origin rpy="0 0 0" xyz="0 0 -0.2"/>
-    <parent link="RR_calf"/>
-    <child link="RR_foot"/>
-  </joint>
-  <link name="RR_foot">
+  <joint name="rr_j3" type="fixed" dont_collapse="true">
+    <origin rpy="0 0 0" xyz="0 0 -0.2"/>
+    <parent link="rr_l2"/>
+    <child link="rr_l3"/>
+  </joint>
+  <link name="rr_l3">
     <visual>
       <origin rpy="0 0 0" xyz="0 0 0"/>
@@ -453,13 +411,13 @@
     </inertial>
   </link>
-  <joint name="RL_hip_joint" type="revolute">
+  <joint name="rl_j0" type="revolute">
     <origin rpy="0 0 0" xyz="-0.183 0.047 0"/>
     <parent link="trunk"/>
-    <child link="RL_hip"/>
+    <child link="rl_l0"/>
     <axis xyz="1 0 0"/>
     <dynamics damping="0" friction="0"/>
     <limit effort="20" lower="-0.802851455917" upper="0.802851455917" velocity="52.4"/>
   </joint>
-  <link name="RL_hip">
+  <link name="rl_l0">
     <visual>
       <origin rpy="0 3.14159265359 0" xyz="0 0 0"/>
@@ -481,27 +439,13 @@
     </inertial>
   </link>
-  <joint name="RL_hip_fixed" type="fixed">
-    <origin rpy="0 0 0" xyz="0 0.081 0"/>
-    <parent link="RL_hip"/>
-    <child link="RL_thigh_shoulder"/>
-  </joint>
-  <!-- this link is only for collision -->
-  <link name="RL_thigh_shoulder">
-    <!-- <collision>
-      <origin rpy="1.57079632679 0 0" xyz="0 0 0"/>
-      <geometry>
-        <cylinder length="0.032" radius="0.041"/>
-      </geometry>
-    </collision> -->
-  </link>
-  <joint name="RL_thigh_joint" type="revolute">
+  <joint name="rl_j1" type="revolute">
     <origin rpy="0 0 0" xyz="0 0.08505 0"/>
-    <parent link="RL_hip"/>
-    <child link="RL_thigh"/>
+    <parent link="rl_l0"/>
+    <child link="rl_l1"/>
     <axis xyz="0 1 0"/>
     <dynamics damping="0" friction="0"/>
     <limit effort="55" lower="-1.0471975512" upper="4.18879020479" velocity="28.6"/>
   </joint>
-  <link name="RL_thigh">
+  <link name="rl_l1">
     <visual>
       <origin rpy="0 0 0" xyz="0 0 0"/>
@@ -523,13 +467,13 @@
     </inertial>
   </link>
-  <joint name="RL_calf_joint" type="revolute">
-    <origin rpy="0 0 0" xyz="0 0 -0.2"/>
-    <parent link="RL_thigh"/>
-    <child link="RL_calf"/>
+  <joint name="rl_j2" type="revolute">
+    <origin rpy="0 0 0" xyz="0 0 -0.2"/>
+    <parent link="rl_l1"/>
+    <child link="rl_l2"/>
     <axis xyz="0 1 0"/>
     <dynamics damping="0" friction="0"/>
     <limit effort="55" lower="-2.69653369433" upper="-0.916297857297" velocity="28.6"/>
   </joint>
-  <link name="RL_calf">
+  <link name="rl_l2">
     <visual>
       <origin rpy="0 0 0" xyz="0 0 0"/>
@@ -551,10 +495,10 @@
     </inertial>
   </link>
-  <joint name="RL_foot_fixed" type="fixed" dont_collapse="true">
-    <origin rpy="0 0 0" xyz="0 0 -0.2"/>
-    <parent link="RL_calf"/>
-    <child link="RL_foot"/>
-  </joint>
-  <link name="RL_foot">
+  <joint name="rl_j3" type="fixed" dont_collapse="true">
+    <origin rpy="0 0 0" xyz="0 0 -0.2"/>
+    <parent link="rl_l2"/>
+    <child link="rl_l3"/>
+  </joint>
+  <link name="rl_l3">
     <visual>
       <origin rpy="0 0 0" xyz="0 0 0"/>

File: meshes/a1/urdf/a1_origin.urdf (robot description, URDF)
Before this commit: robot a1_description, 19 links, 18 joints
Links:
- removed link fl_l0
- removed link fl_l1
- removed link fl_l2
- removed link fl_l3
- removed link fr_l0
- removed link fr_l1
- removed link fr_l2
- removed link fr_l3
- removed link rl_l0
- removed link rl_l1
- removed link rl_l2
- removed link rl_l3
- removed link rr_l0
- removed link rr_l1
- removed link rr_l2
- removed link rr_l3
- added link FL_calf, mass 0.166; collision box size=0.2 0.016 0.016; visual mesh filename=../meshes/calf.dae scale=1 1 1
- added link FL_foot, mass 0.06; collision sphere radius=0.02; visual sphere radius=0.01
- added link FL_hip, mass 0.696; visual mesh filename=../meshes/hip.dae scale=1 1 1
- added link FL_thigh, mass 1.013; collision box size=0.2 0.0245 0.034; visual mesh filename=../meshes/thigh.dae scale=1 1 1
- added link FL_thigh_shoulder
- added link FR_calf, mass 0.166; collision box size=0.2 0.016 0.016; visual mesh filename=../meshes/calf.dae scale=1 1 1
- added link FR_foot, mass 0.06; collision sphere radius=0.02; visual sphere radius=0.01
- added link FR_hip, mass 0.696; visual mesh filename=../meshes/hip.dae scale=1 1 1
- added link FR_thigh, mass 1.013; collision box size=0.2 0.0245 0.034; visual mesh filename=../meshes/thigh_mirror.dae scale=1 1 1
- added link FR_thigh_shoulder
- added link RL_calf, mass 0.166; collision box size=0.2 0.016 0.016; visual mesh filename=../meshes/calf.dae scale=1 1 1
- added link RL_foot, mass 0.06; collision sphere radius=0.02; visual sphere radius=0.01
- added link RL_hip, mass 0.696; visual mesh filename=../meshes/hip.dae scale=1 1 1
- added link RL_thigh, mass 1.013; collision box size=0.2 0.0245 0.034; visual mesh filename=../meshes/thigh.dae scale=1 1 1
- added link RL_thigh_shoulder
- added link RR_calf, mass 0.166; collision box size=0.2 0.016 0.016; visual mesh filename=../meshes/calf.dae scale=1 1 1
- added link RR_foot, mass 0.06; collision sphere radius=0.02; visual sphere radius=0.01
- added link RR_hip, mass 0.696; visual mesh filename=../meshes/hip.dae scale=1 1 1
- added link RR_thigh, mass 1.013; collision box size=0.2 0.0245 0.034; visual mesh filename=../meshes/thigh_mirror.dae scale=1 1 1
- added link RR_thigh_shoulder
Joints:
- removed joint fl_j0
- removed joint fl_j1
- removed joint fl_j2
- removed joint fl_j3
- removed joint fr_j0
- removed joint fr_j1
- removed joint fr_j2
- removed joint fr_j3
- removed joint rl_j0
- removed joint rl_j1
- removed joint rl_j2
- removed joint rl_j3
- removed joint rr_j0
- removed joint rr_j1
- removed joint rr_j2
- removed joint rr_j3
- added joint FL_calf_joint: type revolute, parent FL_thigh, child FL_calf, origin xyz=0 0 -0.2 rpy=0 0 0, axis 0 1 0, limit lower=-2.69653369433 upper=-0.916297857297 effort=55 velocity=28.6
- added joint FL_foot_fixed: type fixed, parent FL_calf, child FL_foot, origin xyz=0 0 -0.2 rpy=0 0 0
- added joint FL_hip_fixed: type fixed, parent FL_hip, child FL_thigh_shoulder, origin xyz=0 0.081 0 rpy=0 0 0
- added joint FL_hip_joint: type revolute, parent trunk, child FL_hip, origin xyz=0.183 0.047 0 rpy=0 0 0, axis 1 0 0, limit lower=-0.802851455917 upper=0.802851455917 effort=20 velocity=52.4
- added joint FL_thigh_joint: type revolute, parent FL_hip, child FL_thigh, origin xyz=0 0.08505 0 rpy=0 0 0, axis 0 1 0, limit lower=-1.0471975512 upper=4.18879020479 effort=55 velocity=28.6
- added joint FR_calf_joint: type revolute, parent FR_thigh, child FR_calf, origin xyz=0 0 -0.2 rpy=0 0 0, axis 0 1 0, limit lower=-2.69653369433 upper=-0.916297857297 effort=55 velocity=28.6
- added joint FR_foot_fixed: type fixed, parent FR_calf, child FR_foot, origin xyz=0 0 -0.2 rpy=0 0 0
- added joint FR_hip_fixed: type fixed, parent FR_hip, child FR_thigh_shoulder, origin xyz=0 -0.081 0 rpy=0 0 0
- added joint FR_hip_joint: type revolute, parent trunk, child FR_hip, origin xyz=0.183 -0.047 0 rpy=0 0 0, axis 1 0 0, limit lower=-0.802851455917 upper=0.802851455917 effort=20 velocity=52.4
- added joint FR_thigh_joint: type revolute, parent FR_hip, child FR_thigh, origin xyz=0 -0.08505 0 rpy=0 0 0, axis 0 1 0, limit lower=-1.0471975512 upper=4.18879020479 effort=55 velocity=28.6
- added joint RL_calf_joint: type revolute, parent RL_thigh, child RL_calf, origin xyz=0 0 -0.2 rpy=0 0 0, axis 0 1 0, limit lower=-2.69653369433 upper=-0.916297857297 effort=55 velocity=28.6
- added joint RL_foot_fixed: type fixed, parent RL_calf, child RL_foot, origin xyz=0 0 -0.2 rpy=0 0 0
- added joint RL_hip_fixed: type fixed, parent RL_hip, child RL_thigh_shoulder, origin xyz=0 0.081 0 rpy=0 0 0
- added joint RL_hip_joint: type revolute, parent trunk, child RL_hip, origin xyz=-0.183 0.047 0 rpy=0 0 0, axis 1 0 0, limit lower=-0.802851455917 upper=0.802851455917 effort=20 velocity=52.4
- added joint RL_thigh_joint: type revolute, parent RL_hip, child RL_thigh, origin xyz=0 0.08505 0 rpy=0 0 0, axis 0 1 0, limit lower=-1.0471975512 upper=4.18879020479 effort=55 velocity=28.6
- added joint RR_calf_joint: type revolute, parent RR_thigh, child RR_calf, origin xyz=0 0 -0.2 rpy=0 0 0, axis 0 1 0, limit lower=-2.69653369433 upper=-0.916297857297 effort=55 velocity=28.6
- added joint RR_foot_fixed: type fixed, parent RR_calf, child RR_foot, origin xyz=0 0 -0.2 rpy=0 0 0
- added joint RR_hip_fixed: type fixed, parent RR_hip, child RR_thigh_shoulder, origin xyz=0 -0.081 0 rpy=0 0 0
- added joint RR_hip_joint: type revolute, parent trunk, child RR_hip, origin xyz=-0.183 -0.047 0 rpy=0 0 0, axis 1 0 0, limit lower=-0.802851455917 upper=0.802851455917 effort=20 velocity=52.4
- added joint RR_thigh_joint: type revolute, parent RR_hip, child RR_thigh, origin xyz=0 -0.08505 0 rpy=0 0 0, axis 0 1 0, limit lower=-1.0471975512 upper=4.18879020479 effort=55 velocity=28.6
