Commit message: add jings pd

File: meshes/wavego_v1/wavego_fix_j0.urdf (robot description, URDF)
Before this commit: robot wavego, 18 links, 17 joints
Links:
- link trunk: mass 0.37688 -> 0.42688

Commit message: fix the bug when effort control pd should be zero

File: meshes/wavego_v1/wavego_fix_j0.urdf (robot description, URDF)
Before this commit: robot wavego, 18 links, 17 joints
Joints:
- joint fl_j0: limit lower=0.0 upper=0.08 effort=55 velocity=10 -> lower=0.0 upper=0.08 effort=0.23 velocity=10
- joint fl_j1: limit lower=-1.570796 upper=0.785398 effort=55 velocity=10 -> lower=-1.570796 upper=0.785398 effort=0.23 velocity=10
- joint fl_j2: limit lower=-0.785398 upper=0.5235988 effort=55 velocity=10 -> lower=-0.785398 upper=0.5235988 effort=0.23 velocity=10
- joint fr_j0: limit lower=0.0 upper=0.08 effort=55 velocity=10 -> lower=0.0 upper=0.08 effort=0.23 velocity=10
- joint fr_j1: limit lower=-1.570796 upper=0.785398 effort=55 velocity=10 -> lower=-1.570796 upper=0.785398 effort=0.23 velocity=10
- joint fr_j2: limit lower=-0.785398 upper=0.5235988 effort=55 velocity=10 -> lower=-0.785398 upper=0.5235988 effort=0.23 velocity=10
- joint rl_j0: limit lower=0.0 upper=0.08 effort=55 velocity=10 -> lower=0.0 upper=0.08 effort=0.23 velocity=10
- joint rl_j1: limit lower=-1.570796 upper=0.785398 effort=55 velocity=10 -> lower=-1.570796 upper=0.785398 effort=0.23 velocity=10
- joint rl_j2: limit lower=-0.785398 upper=0.5235988 effort=55 velocity=10 -> lower=-0.785398 upper=0.5235988 effort=0.23 velocity=10
- joint rr_j0: limit lower=0.0 upper=0.08 effort=55 velocity=10 -> lower=0.0 upper=0.08 effort=0.23 velocity=10
- joint rr_j1: limit lower=-1.570796 upper=0.785398 effort=55 velocity=10 -> lower=-1.570796 upper=0.785398 effort=0.23 velocity=10
- joint rr_j2: limit lower=-0.785398 upper=0.5235988 effort=55 velocity=10 -> lower=-0.785398 upper=0.5235988 effort=0.23 velocity=10
